Commit message: add simulation_rerun package, mac install script, serial transport fixes

File: 3_simulation_rerun/urdf/manipulator.urdf (robot description, URDF)
Before this commit: robot manipulator, 7 links, 6 joints
Links:
- link base_link: geometry collision mesh filename=package://simulation_rerun/meshes/base_link.STL; visual mesh filename=package://simulation_rerun/meshes/base_link.STL
- link claw_left: geometry collision mesh filename=package://simulation_rerun/meshes/claw_left.STL; visual mesh filename=package://simulation_rerun/meshes/claw_left.STL
- link claw_right: geometry collision mesh filename=package://simulation_rerun/meshes/claw_right.STL; visual mesh filename=package://simulation_rerun/meshes/claw_right.STL
- link link_1: geometry collision mesh filename=package://simulation_rerun/meshes/link_1.STL; visual mesh filename=package://simulation_rerun/meshes/link_1.STL
- link link_2: geometry collision mesh filename=package://simulation_rerun/meshes/link_2.STL; visual mesh filename=package://simulation_rerun/meshes/link_2.STL
- link link_3: geometry collision mesh filename=package://simulation_rerun/meshes/link_3.STL; visual mesh filename=package://simulation_rerun/meshes/link_3.STL
